Commit message: move base params changed

File: urdf/servicebot.xacro (robot description, xacro)
@@ -30,5 +30,5 @@
     </link>
     <joint name="laser_joint" type="fixed">
-      <origin xyz="0 0 0.305" rpy="0 0 ${M_PI}"/>
+      <origin xyz="0 0 0.0" rpy="0 0 ${M_PI}"/>
       <parent link="base_link"/>
       <child link="laser"/>
